Commit message: adds the actual fix to tf issues

File: ugv_sim/models/bowser2/model.urdf (robot description, URDF)
Before this commit: robot bowser2, 6 links, 5 joints
Joints:
- removed joint camera_joint
- removed joint front_left_joint
- removed joint front_right_joint
- removed joint imu_joint
- added joint bowser2/camera_joint: type fixed, parent bowser2/base_link, child bowser2/camera_link, origin xyz=0.0   0.0  0.385 rpy=1.5708 3.14159 1.5708, axis 0 1 0, limit lower=0 upper=0 effort=0 velocity=0
- added joint bowser2/front_left_joint: type revolute, parent bowser2/base_link, child bowser2/front_left_wheel, origin xyz=0.3   0.37 -0.05 rpy=0 0 0, axis 0 1 0, limit lower=0 upper=0 effort=0 velocity=0
- added joint bowser2/front_right_joint: type revolute, parent bowser2/base_link, child bowser2/front_right_wheel, origin xyz=0.3  -0.37 -0.05 rpy=0 0 0, axis 0 1 0, limit lower=0 upper=0 effort=0 velocity=0
- added joint bowser2/imu_joint: type fixed, parent bowser2/base_link, child bowser2/imu_link, origin xyz=0 0 0.01
